File: c64converter/board/c64converter.sch (KiCad schematic (older format))
At the start: 38 parts, among them P1 LUMA, P2 LUMA_GND, P3 CHROMA, P4 CHROMA_GND, P5 VIN, P6 VIN_GND, P7 GPIO2, U1 APE8865Y5-30-HF-3, U2 AD9283BRSZ-80, U3 AD9283BRSZ-80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

Commit message: Layout of C64 converter board
Parts:
- D1: footprint (none) -> LEDs:LED_D3.0mm
- OSC1: footprint (none) -> Oscillators:Oscillator_SMD_EuroQuartz_XO53-4pin_5.0x3.2mm_HandSoldering
- S1: footprint (none) -> Housings_DIP:DIP-8_W7.62mm_LongPads
- U1, U4: footprint (none) -> TO_SOT_Packages_SMD:SOT-23-5
- U2, U3: footprint (none) -> Housings_SSOP:SSOP-20_5.3x7.2mm_Pitch0.65mm
- U5: footprint (none) -> Housings_SOIC:SOIC-8_3.9x4.9mm_Pitch1.27mm
Connections:
- net +3V3: no longer U4.3 (~SHDN~)
- net +5V: now also U1.3 (~SHDN~), U4.3 (~SHDN~)
- net 3.0V: no longer U1.3 (~SHDN~)
Changed lines of the file:
@@
 F 0 "U5" H 7100 2900 60  0000 C CNN
 F 1 "THS7316" H 7250 3000 60  0000 C CNN
-F 2 "" H 7250 3000 60  0001 C CNN
+F 2 "Housings_SOIC:SOIC-8_3.9x4.9mm_Pitch1.27mm" H 7250 3000 60  0001 C CNN
 F 3 "" H 7250 3000 60  0001 C CNN
 	1    7250 3000
@@
 F 0 "OSC1" H 5200 2300 60  0000 C CNN
 F 1 "KC7050A80" H 5350 2400 60  0000 C CNN
-F 2 "" H 5350 2350 60  0001 C CNN
+F 2 "Oscillators:Oscillator_SMD_EuroQuartz_XO53-4pin_5.0x3.2mm_HandSoldering" H 5350 2350 60  0001 C CNN
 F 3 "" H 5350 2350 60  0001 C CNN
 	1    5350 2350
@@
 F 0 "U1" H 1800 6100 50  0000 C CNN
 F 1 "APE8865Y5-30-HF-3" H 2100 6050 50  0000 C CNN
-F 2 "" H 2100 5950 50  0000 C CIN
+F 2 "TO_SOT_Packages_SMD:SOT-23-5" H 2100 5950 50  0001 C CIN
 F 3 "" H 2100 5850 50  0000 C CNN
 	1    2100 5850
@@
 F 0 "U4" H 3350 6100 50  0000 C CNN
 F 1 "APE8865Y5-33-HF-3" H 3650 6050 50  0000 C CNN
-F 2 "" H 3650 5950 50  0000 C CIN
+F 2 "TO_SOT_Packages_SMD:SOT-23-5" H 3650 5950 50  0001 C CIN
 F 3 "" H 3650 5850 50  0000 C CNN
 	1    3650 5850
@@
 F 0 "U2" H 3150 2300 60  0000 C CNN
 F 1 "AD9283BRSZ-80" H 3450 2400 60  0000 C CNN
-F 2 "" H 3350 2300 60  0001 C CNN
+F 2 "Housings_SSOP:SSOP-20_5.3x7.2mm_Pitch0.65mm" H 3350 2300 60  0001 C CNN
 F 3 "" H 3350 2300 60  0001 C CNN
 	1    3350 2300
@@
 F 0 "U3" H 3150 4000 60  0000 C CNN
 F 1 "AD9283BRSZ-80" H 3450 4100 60  0000 C CNN
-F 2 "" H 3350 4000 60  0001 C CNN
+F 2 "Housings_SSOP:SSOP-20_5.3x7.2mm_Pitch0.65mm" H 3350 4000 60  0001 C CNN
 F 3 "" H 3350 4000 60  0001 C CNN
 	1    3350 4000
@@
 	3200 5800 3100 5800
 Wire Wire Line
-	3100 5800 3100 5600
+	3100 5600 3100 5950
 Wire Wire Line
 	3650 6150 3650 6500
-Wire Wire Line
-	3200 5950 3150 5950
-Wire Wire Line
-	3150 5950 3150 6200
 Connection ~ 4200 5800
 Wire Wire Line
 	2550 5800 2700 5800
 Wire Wire Line
-	1650 5950 1650 6200
-Wire Wire Line
-	1650 6200 2700 6200
-Wire Wire Line
 	2700 5550 2700 6250
 Wire Wire Line
 	2100 6150 2100 6500
 Wire Wire Line
-	3150 6200 4200 6200
-Wire Wire Line
-	1550 5600 1550 5800
+	1550 5600 1550 5950
 Wire Wire Line
 	1550 5800 1650 5800
@@
 Wire Wire Line
 	2700 6450 2700 6600
-Connection ~ 2700 6200
 Wire Wire Line
 	2100 6500 2700 6500
 Connection ~ 2700 6500
-Connection ~ 4200 6200
 Wire Wire Line
 	3650 6500 4200 6500
@@
 $EndComp
 Wire Wire Line
-	4850 5850 4850 5650
-Wire Wire Line
-	4850 6250 4850 6050
+	4850 5650 4850 5850
+Wire Wire Line
+	4850 6050 4850 6250
 Connection ~ 10700 2350
 Wire Wire Line
@@
 F 0 "S1" H 10200 700 60  0000 C CNN
 F 1 "4_DIP_SWITCH" H 10350 800 60  0000 C CNN
-F 2 "" H 10350 800 60  0001 C CNN
+F 2 "Housings_DIP:DIP-8_W7.62mm_LongPads" H 10350 800 60  0001 C CNN
 F 3 "" H 10350 800 60  0001 C CNN
 	1    10350 800
@@
 F 0 "D1" H 5650 6075 50  0000 L CNN
 F 1 "Power on" H 5525 5850 50  0000 L CNN
-F 2 "" V 5700 5950 50  0001 C CNN
+F 2 "LEDs:LED_D3.0mm" V 5700 5950 50  0001 C CNN
 F 3 "" V 5700 5950 50  0000 C CNN
 	1    5700 5950
@@
 	5700 6150 5700 6050
 Connection ~ 5300 6150
+Wire Wire Line
+	1550 5950 1650 5950
+Connection ~ 1550 5800
+Wire Wire Line
+	3100 5950 3200 5950
+Connection ~ 3100 5800
 $EndSCHEMATC
