File: c64mod/rfreplacement/rfreplacement.sch (KiCad schematic (older format))
At the start: 92 parts, among them U2 10M02SCE144, Y1 Conn_Coaxial

Commit message: rf-replacment: pcb layout
Parts:
- added C30: 10uF, Capacitor_SMD:C_0805_2012Metric_Pad1.15x1.40mm_HandSolder, symbol Device:C_Small
- added SW1: SW_SP3T, footprints:slider, symbol Switch:SW_SP3T
- AMP1, AMP2: footprint Housings_SOIC:SOIC-8_3.9x4.9mm_Pitch1.27mm -> Package_SO:SSOP-8_3.95x5.21x3.27mm_P1.27mm
- C1, C2, C3, C4, C5: footprint Capacitors_SMD:C_0805_HandSoldering -> Capacitor_SMD:C_0805_2012Metric_Pad1.15x1.40mm_HandSolder
- C10, C28, C29: footprint (none) -> Capacitor_SMD:C_0603_1608Metric_Pad1.05x0.95mm_HandSolder
- C11, C12, C13, C14, C15, C16, C17, C18, C19, C20, C21, C22, C23, C24, C25, C26, C27, C31, C32, C33, C34, C6, C7: footprint Capacitors_SMD:C_0603_HandSoldering -> Capacitor_SMD:C_0603_1608Metric_Pad1.05x0.95mm_HandSolder
- C8: footprint (none) -> Capacitor_Tantalum_SMD:CP_EIA-7343-15_Kemet-W_Pad2.25x2.55mm_HandSolder
- C9: footprint (none) -> Capacitor_SMD:C_0805_2012Metric_Pad1.15x1.40mm_HandSolder
- GND1, GND2, GND3, GND4: footprint (none) -> Connector_Pin:Pin_D1.0mm_L10.0mm
- GPIO1: footprint (none) -> Connector_PinHeader_2.54mm:PinHeader_2x10_P2.54mm_Vertical
- GPIO2, JTAG1: footprint (none) -> Connector_PinHeader_2.54mm:PinHeader_2x05_P2.54mm_Vertical
- L1, L2, L3: footprint Capacitors_SMD:C_0805_HandSoldering -> Inductor_SMD:L_0805_2012Metric_Pad1.15x1.40mm_HandSolder
- OSC1: footprint Oscillators:Oscillator_SMD_EuroQuartz_XO53-4pin_5.0x3.2mm_HandSoldering -> Oscillator:Oscillator_SMD_EuroQuartz_XO53-4Pin_5.0x3.2mm_HandSoldering
- PB1, PR1, Y1: footprint (none) -> footprints:RCA_JACK
- R1, R10, R11, R12, R13, R14, R15, R16, R17, R18, R19, R2, R20, R21, R22, R23, R24, R25, R26, R27, R28, R29, R3, R4, R5, R6, R7, R8, R9: footprint Resistors_SMD:R_0805_HandSoldering -> Resistor_SMD:R_0805_2012Metric_Pad1.15x1.40mm_HandSolder
- R30, R31, R32, R33, R34, R35, R36, R37: footprint (none) -> Resistor_SMD:R_0805_2012Metric_Pad1.15x1.40mm_HandSolder
- REG1, REG2: footprint TO_SOT_Packages_SMD:SOT-223 -> Package_TO_SOT_SMD:SOT-223
- RFCON1: footprint (none) -> Connector_PinHeader_2.54mm:PinHeader_1x04_P2.54mm_Vertical
- RFCON2: renamed from JRFCON2; footprint (none) -> Connector_PinHeader_2.54mm:PinHeader_1x04_P2.54mm_Vertical
- RV1: footprint (none) -> Potentiometer_THT:Potentiometer_ACP_CA6-H2,5_Horizontal
Connections:
- net labels added: GNDA, PB, PB1, PR, PR1, PY1, Y
- wire segments 512 -> 520
- no-connect marks 52 -> 53

Commit message: C64 mod: fit rf replacement to long and short main boards
Parts:
- removed RV1: 1k, Potentiometer_THT:Potentiometer_ACP_CA6-H2,5_Horizontal, symbol Device:R_POT
- added GND5, GND6: Conn_01x02, Connector_PinHeader_2.54mm:PinHeader_1x02_P2.54mm_Vertical, symbol Connector_Generic:Conn_01x02
- added JPLUM1: Jumper_2_Open, Connector_PinHeader_2.54mm:PinHeader_1x02_P2.54mm_Vertical, symbol Jumper:Jumper_2_Open
- added R38, R39: 680, Resistor_SMD:R_0805_2012Metric_Pad1.15x1.40mm_HandSolder, symbol Device:R_Small
- added R40: 330, Resistor_SMD:R_0805_2012Metric_Pad1.15x1.40mm_HandSolder, symbol Device:R_Small
- added RFCONC1, RFCONC2: Conn_01x04, Connector_PinHeader_2.54mm:PinHeader_1x04_P2.54mm_Vertical, symbol Connector_Generic:Conn_01x04
- R36: value 150 -> 680
- R37: value 310 -> 330
Connections:
- wire segments 520 -> 540
- no-connect marks 53 -> 54

Commit message: Layout RF replacement board
Parts:
- removed GND6: Conn_01x02, Connector_PinHeader_2.54mm:PinHeader_1x02_P2.54mm_Vertical, symbol Connector_Generic:Conn_01x02
- removed GPIO2: Conn_02x05_Odd_Even, Connector_PinHeader_2.54mm:PinHeader_2x05_P2.54mm_Vertical, symbol Connector_Generic:Conn_02x05_Odd_Even
- removed PB1, PR1, Y1: Conn_Coaxial, footprints:RCA_JACK, symbol Connector:Conn_Coaxial
- added J1: AudioJack4_Ground, footprints:Conrad 4pin audio jack, symbol Connector:AudioJack4_Ground
- C8: footprint Capacitor_Tantalum_SMD:CP_EIA-7343-15_Kemet-W_Pad2.25x2.55mm_HandSolder -> Capacitor_SMD:CP_Elec_6.3x5.8
Connections:
- wire segments 540 -> 507
- no-connect marks 54 -> 60

Commit message: Finished RF replacement  board for C64
Parts:
- JPLUM1: footprint Connector_PinHeader_2.54mm:PinHeader_1x02_P2.54mm_Vertical -> Jumper:SolderJumper-2_P1.3mm_Open_RoundedPad1.0x1.5mm
Changed lines of the file:
@@
 F 0 "JPLUM1" V 3304 5398 50  0000 L CNN
 F 1 "Jumper_2_Open" V 3395 5398 50  0000 L CNN
-F 2 "Connector_PinHeader_2.54mm:PinHeader_1x02_P2.54mm_Vertical" H 3350 5300 50  0001 C CNN
+F 2 "Jumper:SolderJumper-2_P1.3mm_Open_RoundedPad1.0x1.5mm" H 3350 5300 50  0001 C CNN
 F 3 "~" H 3350 5300 50  0001 C CNN
 	1    3350 5300
