File: c64mod/c64board/c64board.sch (KiCad schematic (older format))
At the start: 12 parts, among them J1 Conn_02x10_Odd_Even, U1 VIC-II, U2 MIC5504-3.3YM5, U3 LVC257, U4 LVC245, U5 LVC245

Commit message: Finished C64 mod board
generate gerber files also for Rev. 1
Changed lines of the file:
@@
 EESchema Schematic File Version 4
+LIBS:c64board-cache
 EELAYER 26 0
 EELAYER END
@@
 encoding utf-8
 Sheet 1 1
-Title ""
+Title "C64 mod"
 Date ""
-Rev ""
+Rev "1"
 Comp ""
 Comment1 ""
@@
 L Connector_Generic:Conn_02x10_Odd_Even J1
 U 1 1 5B7FD3C0
-P 8850 3100
-F 0 "J1" H 8900 3717 50  0000 C CNN
-F 1 "Conn_02x10_Odd_Even" H 8900 3626 50  0000 C CNN
-F 2 "Connector_PinHeader_2.54mm:PinHeader_2x10_P2.54mm_Vertical" H 8850 3100 50  0001 C CNN
-F 3 "~" H 8850 3100 50  0001 C CNN
-	1    8850 3100
-	1    0    0    -1
+P 8950 3200
+F 0 "J1" H 9000 3817 50  0000 C CNN
+F 1 "Conn_02x10_Odd_Even" H 9000 3726 50  0000 C CNN
+F 2 "Connector_PinHeader_2.54mm:PinHeader_2x10_P2.54mm_Vertical" H 8950 3200 50  0001 C CNN
+F 3 "~" H 8950 3200 50  0001 C CNN
+	1    8950 3200
+	-1   0    0    1
 $EndComp
 $Comp
@@
 $EndComp
 Wire Wire Line
-	2700 7000 3250 7000
-Wire Wire Line
 	3250 7000 3250 6900
 Wire Wire Line
@@
 Wire Wire Line
 	6100 4850 6200 4850
+Wire Wire Line
+	2650 7000 3250 7000
 $EndSCHEMATC

Commit message: Reverse connector orientation
Changed lines of the file:
@@
 L Connector_Generic:Conn_02x10_Odd_Even J1
 U 1 1 5B7FD3C0
-P 8950 3200
-F 0 "J1" H 9000 3817 50  0000 C CNN
-F 1 "Conn_02x10_Odd_Even" H 9000 3726 50  0000 C CNN
-F 2 "Connector_PinHeader_2.54mm:PinHeader_2x10_P2.54mm_Vertical" H 8950 3200 50  0001 C CNN
-F 3 "~" H 8950 3200 50  0001 C CNN
-	1    8950 3200
-	-1   0    0    1
+P 8850 3100
+F 0 "J1" H 8900 3717 50  0000 C CNN
+F 1 "Conn_02x10_Odd_Even" H 8900 3626 50  0000 C CNN
+F 2 "Connector_PinHeader_2.54mm:PinHeader_2x10_P2.54mm_Vertical" H 8850 3100 50  0001 C CNN
+F 3 "~" H 8850 3100 50  0001 C CNN
+	1    8850 3100
+	1    0    0    -1
 $EndComp
 $Comp
